Commit message: fix joint directions; negate S, R, and T

File: motoman_mh12_support/urdf/mh12_macro.xacro (robot description, xacro)
@@ -106,5 +106,5 @@
     <parent link="${prefix}base_link" />
     <child link="${prefix}link_s" />
-    <axis xyz="0 0 -1" />
+    <axis xyz="0 0 1" />
     <limit  lower="-2.9671" upper="2.9671" effort="0" velocity="3.83972" />
   </joint>
@@ -128,5 +128,5 @@
     <parent link="${prefix}link_u" />
     <child link="${prefix}link_r" />
-    <axis xyz="-1 0 0" />
+    <axis xyz="1 0 0" />
     <limit lower="-3.1416" upper="3.1416" effort="22" velocity="7.15585" />
   </joint>
@@ -143,5 +143,5 @@
     <parent link="${prefix}link_b" />
     <child link="${prefix}link_t" />
-    <axis xyz="-1 0 0" />
+    <axis xyz="1 0 0" />
     <limit lower="-6.2832" upper="6.2832" effort="9.8" velocity="10.647" />
   </joint>

Commit message: add mh12 gazebo support
add initial mh12 gazebo support

Adds inertial tags to support package and initial basic gazebo package

fix moveit controllers config file typo

split arm_controller config files

Allows common parameters to be loaded from this package while joint parameters (with different names) can be swapped out by higher level packages. This is useful when joint names are prefixed by inclusion of the MH12 macro into another robot like YMR12.

move robot plugin out of macro

When multiple robots define a control plugin in their macros and the macros are brought into another robot, there are problems with redefinition of the plugin.

clean up gazebo packages

Fill out manifest and CMakeLists; Clean formatting.

fix formatting in launch file

Cannot break lines in text value of attribute.

add inertia values to mh12 urdf macro

These were computed in from meshlab geometry computation output then scaled by proportion of volume so that the total weight of Base and SLURBT is the advertised 130kg for MH12. The T link had to be scaled up and renormalized because its inertias zeroed out within output precision at normal size.

File: motoman_mh12_support/urdf/mh12_macro.xacro (robot description, xacro)
@@ -8,5 +8,11 @@
   <!-- Links -->
   <link name="${prefix}base_link">
-    <visual>
+    <inertial>
+      <mass value="25.4"/>
+      <origin xyz="-0.057 0.001 0.081" rpy="0 0 0"/>
+      <inertia ixx="0.00462" iyy="0.00769" izz="0.01007" iyz="-0.00005" ixz="0" ixy="0.00003"/>
+    </inertial>
+    <visual>
+      <origin xyz="0 0 0" rpy="0 0 0"/>
       <geometry>
         <mesh filename="package://motoman_mh12_support/meshes/visual/base_link.STL" />
@@ -15,4 +21,5 @@
     </visual>
     <collision>
+      <origin xyz="0 0 0" rpy="0 0 0"/>
       <geometry>
         <mesh filename="package://motoman_mh12_support/meshes/collision/base_link.STL" />
@@ -21,5 +28,11 @@
   </link>
   <link name="${prefix}link_s">
-    <visual>
+    <inertial>
+      <mass value="45.7"/>
+      <origin xyz="0.032 0.015 -0.135" rpy="0 0 0"/>
+      <inertia ixx="0.0284" iyy="0.0324" izz="0.0320" iyz="-0.0021" ixz="-0.0071" ixy="-0.0019"/>
+    </inertial>
+    <visual>
+      <origin xyz="0 0 0" rpy="0 0 0"/>
       <geometry>
         <mesh filename="package://motoman_mh12_support/meshes/visual/link_s.STL" />
@@ -28,4 +41,5 @@
     </visual>
     <collision>
+      <origin xyz="0 0 0" rpy="0 0 0"/>
       <geometry>
         <mesh filename="package://motoman_mh12_support/meshes/collision/link_s.STL" />
@@ -34,5 +48,11 @@
   </link>
   <link name="${prefix}link_l">
-    <visual>
+    <inertial>
+      <mass value="18.1"/>
+      <origin xyz="-0.013 -0.107 0.288" rpy="0 0 0"/>
+      <inertia ixx="0.00970" iyy="0.00992" izz="0.00092" iyz="0.00018" ixz="0.00002" ixy="-0.00013"/>
+    </inertial>
+    <visual>
+      <origin xyz="0 0 0" rpy="0 0 0"/>
       <geometry>
         <mesh filename="package://motoman_mh12_support/meshes/visual/link_l.STL" />
@@ -41,4 +61,5 @@
     </visual>
     <collision>
+      <origin xyz="0 0 0" rpy="0 0 0"/>
       <geometry>
         <mesh filename="package://motoman_mh12_support/meshes/collision/link_l.STL" />
@@ -47,5 +68,11 @@
   </link>
   <link name="${prefix}link_u">
-    <visual>
+    <inertial>
+      <mass value="24.8"/>
+      <origin xyz="0.096 -0.022 0.111" rpy="0 0 0"/>
+      <inertia ixx="0.00668" iyy="0.00696" izz="0.00601" iyz="0.00094" ixz="-0.00214" ixy="0.00055"/>
+    </inertial>
+    <visual>
+      <origin xyz="0 0 0" rpy="0 0 0"/>
       <geometry>
         <mesh filename="package://motoman_mh12_support/meshes/visual/link_u.STL" />
@@ -54,4 +81,5 @@
     </visual>
     <collision>
+      <origin xyz="0 0 0" rpy="0 0 0"/>
       <geometry>
         <mesh filename="package://motoman_mh12_support/meshes/collision/link_u.STL" />
@@ -60,5 +88,11 @@
   </link>
   <link name="${prefix}link_r">
-    <visual>
+    <inertial>
+      <mass value="13.5"/>
+      <origin xyz="0.463 0.002 0.013" rpy="0 0 0"/>
+      <inertia ixx="0.000606" iyy="0.002183" izz="0.002277" iyz="-0.000013" ixz="0" ixy="0.000013"/>
+    </inertial>
+    <visual>
+      <origin xyz="0 0 0" rpy="0 0 0"/>
       <geometry>
         <mesh filename="package://motoman_mh12_support/meshes/visual/link_r.STL" />
@@ -67,4 +101,5 @@
     </visual>
     <collision>
+      <origin xyz="0 0 0" rpy="0 0 0"/>
       <geometry>
         <mesh filename="package://motoman_mh12_support/meshes/collision/link_r.STL" />
@@ -73,5 +108,11 @@
   </link>
   <link name="${prefix}link_b">
-    <visual>
+    <inertial>
+      <mass value="2.37"/>
+      <origin xyz="0.030 -0.001 -0.001" rpy="0 0 0"/>
+      <inertia ixx="0.0000095" iyy="0.0000119" izz="0.0000119" iyz="0" ixz="0" ixy="0"/>
+    </inertial>
+    <visual>
+      <origin xyz="0 0 0" rpy="0 0 0"/>
       <geometry>
         <mesh filename="package://motoman_mh12_support/meshes/visual/link_b.STL" />
@@ -81,4 +122,5 @@
     </visual>
     <collision>
+      <origin xyz="0 0 0" rpy="0 0 0"/>
       <geometry>
         <mesh filename="package://motoman_mh12_support/meshes/collision/link_b.STL" />
@@ -87,5 +129,11 @@
   </link>
   <link name="${prefix}link_t">
-    <visual>
+    <inertial>
+      <mass value="0.118"/>
+      <origin xyz="-0.007 -0.001 0" rpy="0 0 0"/>
+      <inertia ixx="0.0000107" iyy="0.0000055" izz="0.0000055" iyz="0" ixz="0" ixy="0"/>
+    </inertial>
+    <visual>
+      <origin xyz="0 0 0" rpy="0 0 0"/>
       <geometry>
         <mesh filename="package://motoman_mh12_support/meshes/visual/link_t.STL" />
@@ -95,4 +143,5 @@
     </visual>
     <collision>
+      <origin xyz="0 0 0" rpy="0 0 0"/>
       <geometry>
         <mesh filename="package://motoman_mh12_support/meshes/collision/link_t.STL" />
@@ -103,49 +152,53 @@
   <!-- JOINTS -->
   <joint name="${prefix}joint_s" type="revolute">
-    <origin xyz="0 0 0.45"/>
+    <origin xyz="0 0 0.45" rpy="0 0 0"/>
     <parent link="${prefix}base_link" />
     <child link="${prefix}link_s" />
     <axis xyz="0 0 1" />
     <limit  lower="-2.9671" upper="2.9671" effort="0" velocity="3.83972" />
+    <dynamics damping="0.0" friction="0.0"/>
   </joint>
   <joint name="${prefix}joint_l" type="revolute">
-    <origin xyz="0.155 0 0"/>
+    <origin xyz="0.155 0 0" rpy="0 0 0"/>
     <parent link="${prefix}link_s" />
     <child link="${prefix}link_l" />
     <axis xyz="0 -1 0" />
     <limit lower="-1.5708" upper="2.7053" effort="0" velocity="3.49066" />
+    <dynamics damping="0.0" friction="0.0"/>
   </joint>
   <joint name="${prefix}joint_u" type="revolute">
-    <origin
-      xyz="0 0 0.614"/>
+    <origin xyz="0 0 0.614" rpy="0 0 0"/>
     <parent link="${prefix}link_l" />
     <child link="${prefix}link_u" />
     <axis xyz="0 -1 0" />
     <limit lower="-3.0543" upper="4.1888" effort="0" velocity="3.8397" />
+    <dynamics damping="0.0" friction="0.0"/>
   </joint>
   <joint name="${prefix}joint_r" type="revolute">
-    <origin xyz="0 0 0.2"/>
+    <origin xyz="0 0 0.2" rpy="0 0 0"/>
     <parent link="${prefix}link_u" />
     <child link="${prefix}link_r" />
     <axis xyz="1 0 0" />
     <limit lower="-3.1416" upper="3.1416" effort="22" velocity="7.15585" />
+    <dynamics damping="0.0" friction="0.0"/>
   </joint>
   <joint name="${prefix}joint_b" type="revolute">
-    <origin
-      xyz="0.64 0 0"/>
+    <origin xyz="0.64 0 0" rpy="0 0 0"/>
     <parent link="${prefix}link_r" />
     <child link="${prefix}link_b" />
     <axis xyz="0 -1 0" />
     <limit lower="-2.3562" upper="2.3562" effort="22" velocity="7.15585" />
+    <dynamics damping="0.0" friction="0.0"/>
   </joint>
   <joint name="${prefix}joint_t" type="revolute">
-    <origin xyz="0.1 0 0"/>
+    <origin xyz="0.1 0 0" rpy="0 0 0"/>
     <parent link="${prefix}link_b" />
     <child link="${prefix}link_t" />
     <axis xyz="1 0 0" />
     <limit lower="-6.2832" upper="6.2832" effort="9.8" velocity="10.647" />
+    <dynamics damping="0.0" friction="0.0"/>
   </joint>
   <joint name="${prefix}link_t-tool0" type="fixed">
-    <origin rpy="0 1.5708 0"/>
+    <origin xyz="0 0 0" rpy="0 1.5708 0"/>
     <parent link="${prefix}link_t"/>
     <child link="${prefix}tool0"/>

Commit message: fix mh12 packages for motoros functionality
fix mh12 joint directions for LRT

The joint directions for L, R, and T are labeled correctly on the arm. This contradicts previous information received from the software groups and MotoSim

load mh12 joint names unless sim

fix mh12 real controller namespace

fix mh12 urdf joint limits

This resolves problems in failing to reach poses outside the previous position limits (upper and lower) for joint_u. The replacement values came from a URDF provided by Bill Edwards in an email on 4/5/2018. These new limits also include velocity and effort for every link.

update mh12 moveit config poses

fix half pi values

File: motoman_mh12_support/urdf/mh12_macro.xacro (robot description, xacro)
@@ -4,5 +4,5 @@
   <!-- Properties -->
   <material name="mh12_deep_blue">
-        <color rgba="0.12941 0.14902 0.74902 1" />
+        <color rgba="0.12941 0.14902 0.74902 1"/>
   </material>
   <!-- Links -->
@@ -16,12 +16,12 @@
       <origin xyz="0 0 0" rpy="0 0 0"/>
       <geometry>
-        <mesh filename="package://motoman_mh12_support/meshes/visual/base_link.STL" />
-      </geometry>
-      <material name="mh12_deep_blue"/>
-    </visual>
-    <collision>
-      <origin xyz="0 0 0" rpy="0 0 0"/>
-      <geometry>
-        <mesh filename="package://motoman_mh12_support/meshes/collision/base_link.STL" />
+        <mesh filename="package://motoman_mh12_support/meshes/visual/base_link.STL"/>
+      </geometry>
+      <material name="mh12_deep_blue"/>
+    </visual>
+    <collision>
+      <origin xyz="0 0 0" rpy="0 0 0"/>
+      <geometry>
+        <mesh filename="package://motoman_mh12_support/meshes/collision/base_link.STL"/>
       </geometry>
     </collision>
@@ -36,12 +36,12 @@
       <origin xyz="0 0 0" rpy="0 0 0"/>
       <geometry>
-        <mesh filename="package://motoman_mh12_support/meshes/visual/link_s.STL" />
-      </geometry>
-      <material name="mh12_deep_blue"/>
-    </visual>
-    <collision>
-      <origin xyz="0 0 0" rpy="0 0 0"/>
-      <geometry>
-        <mesh filename="package://motoman_mh12_support/meshes/collision/link_s.STL" />
+        <mesh filename="package://motoman_mh12_support/meshes/visual/link_s.STL"/>
+      </geometry>
+      <material name="mh12_deep_blue"/>
+    </visual>
+    <collision>
+      <origin xyz="0 0 0" rpy="0 0 0"/>
+      <geometry>
+        <mesh filename="package://motoman_mh12_support/meshes/collision/link_s.STL"/>
       </geometry>
     </collision>
@@ -56,12 +56,12 @@
       <origin xyz="0 0 0" rpy="0 0 0"/>
       <geometry>
-        <mesh filename="package://motoman_mh12_support/meshes/visual/link_l.STL" />
-      </geometry>
-      <material name="mh12_deep_blue"/>
-    </visual>
-    <collision>
-      <origin xyz="0 0 0" rpy="0 0 0"/>
-      <geometry>
-        <mesh filename="package://motoman_mh12_support/meshes/collision/link_l.STL" />
+        <mesh filename="package://motoman_mh12_support/meshes/visual/link_l.STL"/>
+      </geometry>
+      <material name="mh12_deep_blue"/>
+    </visual>
+    <collision>
+      <origin xyz="0 0 0" rpy="0 0 0"/>
+      <geometry>
+        <mesh filename="package://motoman_mh12_support/meshes/collision/link_l.STL"/>
       </geometry>
     </collision>
@@ -76,12 +76,12 @@
       <origin xyz="0 0 0" rpy="0 0 0"/>
       <geometry>
-        <mesh filename="package://motoman_mh12_support/meshes/visual/link_u.STL" />
-      </geometry>
-      <material name="mh12_deep_blue"/>
-    </visual>
-    <collision>
-      <origin xyz="0 0 0" rpy="0 0 0"/>
-      <geometry>
-        <mesh filename="package://motoman_mh12_support/meshes/collision/link_u.STL" />
+        <mesh filename="package://motoman_mh12_support/meshes/visual/link_u.STL"/>
+      </geometry>
+      <material name="mh12_deep_blue"/>
+    </visual>
+    <collision>
+      <origin xyz="0 0 0" rpy="0 0 0"/>
+      <geometry>
+        <mesh filename="package://motoman_mh12_support/meshes/collision/link_u.STL"/>
       </geometry>
     </collision>
@@ -96,12 +96,12 @@
       <origin xyz="0 0 0" rpy="0 0 0"/>
       <geometry>
-        <mesh filename="package://motoman_mh12_support/meshes/visual/link_r.STL" />
-      </geometry>
-      <material name="mh12_deep_blue"/>
-    </visual>
-    <collision>
-      <origin xyz="0 0 0" rpy="0 0 0"/>
-      <geometry>
-        <mesh filename="package://motoman_mh12_support/meshes/collision/link_r.STL" />
+        <mesh filename="package://motoman_mh12_support/meshes/visual/link_r.STL"/>
+      </geometry>
+      <material name="mh12_deep_blue"/>
+    </visual>
+    <collision>
+      <origin xyz="0 0 0" rpy="0 0 0"/>
+      <geometry>
+        <mesh filename="package://motoman_mh12_support/meshes/collision/link_r.STL"/>
       </geometry>
     </collision>
@@ -116,5 +116,5 @@
       <origin xyz="0 0 0" rpy="0 0 0"/>
       <geometry>
-        <mesh filename="package://motoman_mh12_support/meshes/visual/link_b.STL" />
+        <mesh filename="package://motoman_mh12_support/meshes/visual/link_b.STL"/>
       </geometry>
       <material name="mh12_deep_blue">
@@ -124,5 +124,5 @@
       <origin xyz="0 0 0" rpy="0 0 0"/>
       <geometry>
-        <mesh filename="package://motoman_mh12_support/meshes/collision/link_b.STL" />
+        <mesh filename="package://motoman_mh12_support/meshes/collision/link_b.STL"/>
       </geometry>
     </collision>
@@ -137,5 +137,5 @@
       <origin xyz="0 0 0" rpy="0 0 0"/>
       <geometry>
-        <mesh filename="package://motoman_mh12_support/meshes/visual/link_t.STL" />
+        <mesh filename="package://motoman_mh12_support/meshes/visual/link_t.STL"/>
       </geometry>
       <material name="mh12_deep_blue">
@@ -145,5 +145,5 @@
       <origin xyz="0 0 0" rpy="0 0 0"/>
       <geometry>
-        <mesh filename="package://motoman_mh12_support/meshes/collision/link_t.STL" />
+        <mesh filename="package://motoman_mh12_support/meshes/collision/link_t.STL"/>
       </geometry>
     </collision>
@@ -153,48 +153,48 @@
   <joint name="${prefix}joint_s" type="revolute">
     <origin xyz="0 0 0.45" rpy="0 0 0"/>
-    <parent link="${prefix}base_link" />
-    <child link="${prefix}link_s" />
-    <axis xyz="0 0 1" />
-    <limit  lower="-2.9671" upper="2.9671" effort="0" velocity="3.83972" />
+    <parent link="${prefix}base_link"/>
+    <child link="${prefix}link_s"/>
+    <axis xyz="0 0 1"/>
+    <limit lower="-2.9670" upper="2.9670" effort="648.27" velocity="3.8397"/>
     <dynamics damping="0.0" friction="0.0"/>
   </joint>
   <joint name="${prefix}joint_l" type="revolute">
     <origin xyz="0.155 0 0" rpy="0 0 0"/>
-    <parent link="${prefix}link_s" />
-    <child link="${prefix}link_l" />
-    <axis xyz="0 -1 0" />
-    <limit lower="-1.5708" upper="2.7053" effort="0" velocity="3.49066" />
+    <parent link="${prefix}link_s"/>
+    <child link="${prefix}link_l"/>
+    <axis xyz="0 1 0"/>
+    <limit lower="-1.5708" upper="2.7052" effort="874.65" velocity="3.4906"/>
     <dynamics damping="0.0" friction="0.0"/>
   </joint>
   <joint name="${prefix}joint_u" type="revolute">
     <origin xyz="0 0 0.614" rpy="0 0 0"/>
-    <parent link="${prefix}link_l" />
-    <child link="${prefix}link_u" />
-    <axis xyz="0 -1 0" />
-    <limit lower="-3.0543" upper="4.1888" effort="0" velocity="3.8397" />
+    <parent link="${prefix}link_l"/>
+    <child link="${prefix}link_u"/>
+    <axis xyz="0 -1 0"/>
+    <limit lower="-1.4835" upper="2.6179" effort="257.25" velocity="3.8397"/>
     <dynamics damping="0.0" friction="0.0"/>
   </joint>
   <joint name="${prefix}joint_r" type="revolute">
     <origin xyz="0 0 0.2" rpy="0 0 0"/>
-    <parent link="${prefix}link_u" />
-    <child link="${prefix}link_r" />
-    <axis xyz="1 0 0" />
-    <limit lower="-3.1416" upper="3.1416" effort="22" velocity="7.15585" />
+    <parent link="${prefix}link_u"/>
+    <child link="${prefix}link_r"/>
+    <axis xyz="-1 0 0"/>
+    <limit lower="-3.1415" upper="3.1415" effort="74.97" velocity="7.1558"/>
     <dynamics damping="0.0" friction="0.0"/>
   </joint>
   <joint name="${prefix}joint_b" type="revolute">
     <origin xyz="0.64 0 0" rpy="0 0 0"/>
-    <parent link="${prefix}link_r" />
-    <child link="${prefix}link_b" />
-    <axis xyz="0 -1 0" />
-    <limit lower="-2.3562" upper="2.3562" effort="22" velocity="7.15585" />
+    <parent link="${prefix}link_r"/>
+    <child link="${prefix}link_b"/>
+    <axis xyz="0 -1 0"/>
+    <limit lower="-2.3562" upper="2.3562" effort="44.69" velocity="7.1558"/>
     <dynamics damping="0.0" friction="0.0"/>
   </joint>
   <joint name="${prefix}joint_t" type="revolute">
     <origin xyz="0.1 0 0" rpy="0 0 0"/>
-    <parent link="${prefix}link_b" />
-    <child link="${prefix}link_t" />
-    <axis xyz="1 0 0" />
-    <limit lower="-6.2832" upper="6.2832" effort="9.8" velocity="10.647" />
+    <parent link="${prefix}link_b"/>
+    <child link="${prefix}link_t"/>
+    <axis xyz="-1 0 0"/>
+    <limit lower="-6.2832" upper="6.2832" effort="14.80" velocity="10.6465"/>
     <dynamics damping="0.0" friction="0.0"/>
   </joint>
